Commit message: aroco description : update xacro files

File: aroco_description/urdf/aroco.urdf.xacro (robot description, xacro)
@@ -4,6 +4,6 @@
   <xacro:arg name="mode" default="simulation" />
   <xacro:arg name="controller_conf_yaml_file" default=""/>
-  <xacro:include filename="$(find adap2e_description)/urdf/aroco.xacro" />
-  <xacro:adap2e model="slim" mode="$(arg mode)" prefix="$(arg prefix)"/>
+  <xacro:include filename="$(find aroco_description)/urdf/aroco.xacro" />
+  <xacro:aroco mode="$(arg mode)" prefix="$(arg prefix)"/>
   <gazebo>
     <plugin filename="libgazebo_ros2_control.so" name="gazebo_ros2_control">

File: aroco_description/urdf/aroco.xacro (robot description, xacro)
@@ -1,7 +1,7 @@
 <?xml version="1.0"?>
-<robot name="adap2e" xmlns:xacro="http://www.ros.org/wiki/xacro">
+<robot name="aroco" xmlns:xacro="http://www.ros.org/wiki/xacro">
     <xacro:include filename="$(find romea_mobile_base_description)/urdf/2AS_4WD_chassis.xacro" />
     <xacro:include filename="$(find romea_mobile_base_description)/ros2_control/2AS_4WD.ros2_control.xacro"/>
-    <xacro:property name="conf" value="$(find adap2e_description)/config/aroco.yaml" />
+    <xacro:property name="conf" value="$(find aroco_description)/config/aroco.yaml" />
     <xacro:property name="props" value="${load_yaml(conf)['/**']['ros__parameters']['base_info']}" />
     <!-- Link names -->
@@ -21,7 +21,7 @@
     <!-- Joint names -->
     <xacro:property name="base_footprint_joint" value="${props['joints']['base_footprint_joint_name']}" />
-    <xacro:property name="front_axle_steering_joint" value="${props['links']['front_axle_steering_joint_name']}" />
-    <xacro:property name="rear_axle_steering_joint" value="${props['links']['rear_axle_steering_joint_name']}" />
     <xacro:property name="inertial_joint" value="${props['joints']['inertial_joint_name']}" />
+    <xacro:property name="front_axle_steering_joint" value="${props['joints']['front_axle_steering_joint_name']}" />
+    <xacro:property name="rear_axle_steering_joint" value="${props['joints']['rear_axle_steering_joint_name']}" />
     <xacro:property name="front_left_wheel_steering_joint" value="${props['joints']['front_left_wheel_steering_joint_name']}" />
     <xacro:property name="front_right_wheel_steering_joint" value="${props['joints']['front_right_wheel_steering_joint_name']}" />
@@ -43,8 +43,8 @@
     <xacro:property name="mass_center_y" value="${props['inertia']['center'][1]}" />
     <xacro:property name="mass_center_z" value="${props['inertia']['center'][2]}" />
-    <xacro:property name="minimal_axle_steering_angle" value="-${props['axles_steering_control']['command']['maximal_angle']}"/>
     <xacro:property name="maximal_axle_steering_angle" value="${props['axles_steering_control']['command']['maximal_angle']}"/>
-    <xacro:property name="minimal_wheel_steering_angle" value="-${props['axles_steering_control']['command']['maximal_angle']}"/>
-    <xacro:property name="maximal_wheel_steering_angle" value="${props['axles_steering_control']['command']['maximal_angle']}"/>
+    <xacro:property name="maximal_wheel_steering_angle" value="${atan(tan(maximal_axle_steering_angle)/(1-tan(maximal_axle_steering_angle)*front_track/(2*wheelbase)))}"/>
+    <xacro:property name="minimal_axle_steering_angle" value="${-maximal_axle_steering_angle}"/>
+    <xacro:property name="minimal_wheel_steering_angle" value="${-maximal_wheel_steering_angle} "/>
     <xacro:property name="maximal_wheel_speed" value="${props['wheels_speed_control']['command']['maximal_speed']}"/>
     <xacro:property name="body_reference_x" value="${props['control_point'][0]}" />
@@ -66,5 +66,5 @@
     <!-- Ros2 control hardware plugin -->
     <xacro:property name="simulation_hardware_plugin" value="romea_mobile_base_gazebo/GazeboSystemInterface2AS4WD"/>
-    <xacro:property name="live_hardware_plugin" value="adap2e_hardware/ArocoHardware"/>
+    <xacro:property name="live_hardware_plugin" value="aroco_hardware/ArocoHardware"/>
     <xacro:macro name="aroco" params="mode prefix">
       <!-- visual chassis -->

Commit message: split ros2_control from urdf description remove robot state publisher from launch files

File: aroco_description/urdf/aroco.urdf.xacro (robot description, xacro)
@@ -3,15 +3,16 @@
   <xacro:arg name="prefix" default="aroco_" />
   <xacro:arg name="mode" default="simulation" />
-  <xacro:arg name="controller_conf_yaml_file" default="" />
+  <xacro:arg name="base_name" default="base" />
+  <xacro:arg name="ros2_control_config_urdf_file" default="" />
+  <xacro:arg name="controller_manager_config_yaml_file" default="" />
   <xacro:arg name="ros_prefix" default="/aroco/" />
   <xacro:include filename="$(find aroco_description)/urdf/aroco.xacro" />
   <xacro:aroco mode="$(arg mode)" prefix="$(arg prefix)" />
   <gazebo>
-    <plugin filename="libgazebo_ros2_control.so" name="gazebo_ros2_control">
-      <hardware>$(arg prefix)base</hardware>
-      <robot_param_node>$(arg ros_prefix)robot_state_publisher</robot_param_node>
-      <parameters>$(arg controller_conf_yaml_file)</parameters>
+    <plugin filename="libromea_gazebo_ros2_control.so" name="gazebo_ros2_control">
+      <ros2_control_config_file>$(arg ros2_control_config_urdf_file)</ros2_control_config_file>
+      <controller_manager_config_file>$(arg controller_manager_config_yaml_file)</controller_manager_config_file>
       <ros>
-        <namespace>$(arg ros_prefix)base</namespace>
+        <namespace>$(arg ros_prefix)$(arg base_name)</namespace>
       </ros>
     </plugin>

File: aroco_description/urdf/aroco.xacro (robot description, xacro)
@@ -2,6 +2,4 @@
 <robot name="aroco" xmlns:xacro="http://www.ros.org/wiki/xacro">
   <xacro:include filename="$(find romea_mobile_base_description)/urdf/base2ASxxx.chassis.xacro" />
-  <xacro:include
-    filename="$(find romea_mobile_base_description)/ros2_control/base2AS4WD.ros2_control.xacro" />
   <xacro:property name="conf" value="$(find aroco_description)/config/aroco.yaml" />
   <xacro:property name="props" value="${load_yaml(conf)}" />
@@ -98,8 +96,4 @@
     value="${props['geometry']['rear_axle']['wheels']['hub_carrier_offset']}" />
   <xacro:property name="chassis_height" value="${min(front_wheel_radius,rear_wheel_radius)}" />
-  <!-- Ros2 control hardware plugin -->
-  <xacro:property name="simulation_hardware_plugin"
-    value="romea_mobile_base_gazebo/GazeboSystemInterface2AS4WD" />
-  <xacro:property name="live_hardware_plugin" value="aroco_hardware/ArocoHardware" />
   <xacro:macro name="aroco" params="mode prefix">
     <!-- visual chassis -->
@@ -118,7 +112,4 @@
       <mesh filename="package://aroco_description/meshes/wheel.dae" />
     </xacro:chassis>
-    <xacro:if value="${mode == 'simulation' or mode == 'live'}">
-      <xacro:base_control mode="${mode}" />
-    </xacro:if>
   </xacro:macro>
 </robot>
