Commit message: description: update xacro file
Signed-off-by: Jean Laneurit <jean.laneurit@inrae.fr>

File: aroco_description/urdf/aroco.xacro (robot description, xacro)
@@ -5,7 +5,10 @@
   <xacro:property name="props" value="${load_yaml(conf)}" />
   <!-- Link names -->
-  <xacro:property name="base_link" value="${props['links']['base_link_name']}" />
-  <xacro:property name="base_footprint_link" value="${props['links']['base_footprint_link_name']}" />
-  <xacro:property name="inertial_link" value="${props['links']['inertial_link_name']}" />
+  <xacro:property name="base_link"
+    value="${props['links']['base_link_name']}" />
+  <xacro:property name="base_footprint_link"
+    value="${props['links']['base_footprint_link_name']}" />
+  <xacro:property name="inertial_link"
+    value="${props['links']['inertial_link_name']}" />
   <xacro:property name="front_axle_steering_link"
     value="${props['links']['front_axle_steering_link_name']}" />
@@ -31,5 +34,6 @@
   <xacro:property name="base_footprint_joint"
     value="${props['joints']['base_footprint_joint_name']}" />
-  <xacro:property name="inertial_joint" value="${props['joints']['inertial_joint_name']}" />
+  <xacro:property name="inertial_joint"
+    value="${props['joints']['inertial_joint_name']}" />
   <xacro:property name="front_axle_steering_joint"
     value="${props['joints']['front_axle_steering_joint_name']}" />
@@ -53,30 +57,39 @@
     value="${props['joints']['rear_right_wheel_spinning_joint_name']}" />
   <!-- Base Properties -->
-  <xacro:property name="aabb_length" value="${props['geometry']['aabb']['length']}" />
-  <xacro:property name="aabb_width" value="${props['geometry']['aabb']['width']}" />
-  <xacro:property name="aabb_height" value="${props['geometry']['aabb']['height']}" />
-  <xacro:property name="aabb_center_x" value="${props['geometry']['aabb']['center'][0]}" />
-  <xacro:property name="aabb_center_y" value="${props['geometry']['aabb']['center'][1]}" />
-  <xacro:property name="aabb_center_z" value="${props['geometry']['aabb']['center'][2]}" />
-  <xacro:property name="wheelbase" value="${props['geometry']['axles_distance']}" />
-  <xacro:property name="front_track" value="${props['geometry']['front_axle']['wheels_distance']}" />
-  <xacro:property name="rear_track" value="${props['geometry']['rear_axle']['wheels_distance']}" />
-  <xacro:property name="mass_base" value="${props['inertia']['mass']}" />
-  <xacro:property name="mass_center_x" value="${props['inertia']['center'][0]}" />
-  <xacro:property name="mass_center_y" value="${props['inertia']['center'][1]}" />
-  <xacro:property name="mass_center_z" value="${props['inertia']['center'][2]}" />
-  <xacro:property name="maximal_axle_steering_angle"
-    value="${props['axles_steering_control']['command']['maximal_angle']}" />
-  <xacro:property name="maximal_wheel_steering_angle"
-    value="${atan(tan(maximal_axle_steering_angle)/(1-tan(maximal_axle_steering_angle)*front_track/(2*wheelbase)))}" />
-  <xacro:property name="minimal_axle_steering_angle" value="${-maximal_axle_steering_angle}" />
-  <xacro:property name="minimal_wheel_steering_angle" value="${-maximal_wheel_steering_angle} " />
-  <xacro:property name="maximal_wheel_speed"
-    value="${props['wheels_speed_control']['command']['maximal_speed']}" />
-  <xacro:property name="body_reference_x" value="${props['control_point'][0]}" />
+  <xacro:property name="aabb_length"
+    value="${props['geometry']['aabb']['length']}" />
+  <xacro:property name="aabb_width"
+    value="${props['geometry']['aabb']['width']}" />
+  <xacro:property name="aabb_height"
+    value="${props['geometry']['aabb']['height']}" />
+  <xacro:property name="aabb_center_x"
+    value="${props['geometry']['aabb']['center'][0]}" />
+  <xacro:property name="aabb_center_y"
+    value="${props['geometry']['aabb']['center'][1]}" />
+  <xacro:property name="aabb_center_z"
+    value="${props['geometry']['aabb']['center'][2]}" />
+  <xacro:property name="wheelbase"
+    value="${props['geometry']['axles_distance']}" />
+  <xacro:property name="front_track"
+    value="${props['geometry']['front_axle']['wheels_distance']}" />
+  <xacro:property name="rear_track"
+    value="${props['geometry']['rear_axle']['wheels_distance']}" />
+  <xacro:property name="mass_base"
+    value="${props['inertia']['mass']}" />
+  <xacro:property name="mass_center_x"
+    value="${props['inertia']['center'][0]}" />
+  <xacro:property name="mass_center_y"
+    value="${props['inertia']['center'][1]}" />
+  <xacro:property name="mass_center_z"
+    value="${props['inertia']['center'][2]}" />
+  <xacro:property name="body_reference_x"
+    value="${props['control_point'][0]}" />
+ <xacro:property name="ground_clearance"
+    value="${props['geometry']['ground_clearance']}" />
   <!-- Wheel Properties -->
-  <xacro:property name="steering_link_mass" value="30" />
-  <xacro:property name="steering_link_y" value="0.05" />
-  <xacro:property name="steering_link_xz" value="0.1" />
+  <xacro:property name="front_hub_carrier_offset"
+    value="${props['geometry']['front_axle']['wheels']['hub_carrier_offset']}" />
+  <xacro:property name="rear_hub_carrier_offset"
+    value="${props['geometry']['rear_axle']['wheels']['hub_carrier_offset']}" />
   <xacro:property name="front_wheel_radius"
     value="${props['geometry']['front_axle']['wheels']['radius']}" />
@@ -87,15 +100,29 @@
   <xacro:property name="rear_wheel_width"
     value="${props['geometry']['rear_axle']['wheels']['width']}" />
+  <xacro:property name="chassis_height"
+    value="${min(front_wheel_radius,rear_wheel_radius)}" />
+  <xacro:property name="maximal_wheel_speed"
+    value="${props['wheels_speed_control']['command']['maximal_speed']}" />
   <xacro:property name="front_wheel_mass" value="10" />
   <xacro:property name="rear_wheel_mass" value="10" />
-  <!-- Wheel Mounting Positions -->
-  <xacro:property name="ground_clearance"
-    value="${props['geometry']['ground_clearance']}" />
-  <xacro:property name="front_wheel_y_offset"
-    value="${props['geometry']['front_axle']['wheels']['hub_carrier_offset']}" />
-  <xacro:property name="rear_wheel_y_offset"
-    value="${props['geometry']['rear_axle']['wheels']['hub_carrier_offset']}" />
-  <xacro:property name="chassis_height"
-    value="${min(front_wheel_radius,rear_wheel_radius)}" />
+  <!-- Steering Properties -->
+  <xacro:property name="maximal_axle_steering_angle"
+    value="${props['axles_steering_control']['command']['maximal_angle']}" />
+  <xacro:property name="maximal_wheel_steering_angle"
+    value="${atan(tan(maximal_axle_steering_angle)/(1-tan(maximal_axle_steering_angle)*front_track/(2*wheelbase)))}" />
+  <xacro:property name="minimal_axle_steering_angle"
+    value="${-maximal_axle_steering_angle}" />
+  <xacro:property name="minimal_wheel_steering_angle"
+    value="${-maximal_wheel_steering_angle} " />
+  <xacro:property name="front_axle_steering_link_mass" value="1" />
+  <xacro:property name="front_axle_steering_link_x" value="0.05" />
+  <xacro:property name="front_axle_steering_link_y" value="0.05" />
+  <xacro:property name="front_axle_steering_link_z" value="0.05" />
+  <xacro:property name="front_wheel_steering_link_mass" value="30" />
+  <xacro:property name="front_wheel_steering_link_y" value="${front_hub_carrier_offset}" />
+  <xacro:property name="front_wheel_steering_link_xz" value="0.05" />
+  <xacro:property name="rear_wheel_steering_link_mass" value="30" />
+  <xacro:property name="rear_wheel_steering_link_y" value="${front_hub_carrier_offset}" />
+  <xacro:property name="rear_wheel_steering_link_xz" value="0.05" />
   <xacro:macro name="aroco" params="mode prefix">
     <!-- visual chassis -->
@@ -109,7 +136,11 @@
         </geometry>
       </visual>
-      <!-- visual steering -->
+      <!-- visual front steering -->
       <mesh filename="package://aroco_description/meshes/wheel_steered.dae" />
-      <!-- visual wheel -->
+      <!-- visual rear steering -->
+      <mesh filename="package://aroco_description/meshes/wheel_steered.dae" />
+      <!-- visual front wheel -->
+      <mesh filename="package://aroco_description/meshes/wheel.dae" />
+      <!-- visual rear wheel -->
       <mesh filename="package://aroco_description/meshes/wheel.dae" />
     </xacro:chassis>

Commit message: refactoring of yaml and xacro files
Signed-off-by: jean.laneurit <jean.laneurit@inrae.fr>

File: aroco_description/urdf/aroco.xacro (robot description, xacro)
@@ -85,5 +85,5 @@
   <xacro:property name="body_reference_x"
     value="${props['control_point'][0]}" />
- <xacro:property name="ground_clearance"
+  <xacro:property name="ground_clearance"
     value="${props['geometry']['ground_clearance']}" />
   <!-- Wheel Properties -->

Commit message: description: change way to define visual in xacro file
Signed-off-by: jean.laneurit <jean.laneurit@inrae.fr>

File: aroco_description/urdf/aroco.xacro (robot description, xacro)
@@ -2,4 +2,7 @@
 <robot name="aroco" xmlns:xacro="http://www.ros.org/wiki/xacro">
   <xacro:include filename="$(find romea_mobile_base_description)/urdf/base2ASxxx.chassis.xacro" />
+  <xacro:include filename="$(find aroco_description)/urdf/visual/chassis.xacro" />
+  <xacro:include filename="$(find aroco_description)/urdf/visual/wheels.xacro" />
+  <xacro:include filename="$(find aroco_description)/urdf/visual/arms.xacro" />
   <xacro:property name="conf" value="$(find aroco_description)/config/aroco.yaml" />
   <xacro:property name="props" value="${load_yaml(conf)}" />
@@ -88,4 +91,6 @@
     value="${props['geometry']['ground_clearance']}" />
   <!-- Wheel Properties -->
+  <xacro:property name="front_wheel_x_offset" value="0.0" />
+  <xacro:property name="rear_wheel_x_offset" value="0.0" />
   <xacro:property name="front_hub_carrier_offset"
     value="${props['geometry']['front_axle']['wheels']['hub_carrier_offset']}" />
@@ -123,25 +128,17 @@
   <xacro:property name="front_wheel_steering_link_xz" value="0.05" />
   <xacro:property name="rear_wheel_steering_link_mass" value="30" />
-  <xacro:property name="rear_wheel_steering_link_y" value="${front_hub_carrier_offset}" />
+  <xacro:property name="rear_wheel_steering_link_y" value="${rear_hub_carrier_offset}" />
   <xacro:property name="rear_wheel_steering_link_xz" value="0.05" />
   <xacro:macro name="aroco" params="mode prefix">
-    <!-- visual chassis -->
     <xacro:chassis>
-      <!-- visual chassis -->
-      <visual>
-        <origin xyz="${0.03-body_reference_x} 0 ${chassis_height-aabb_height/2}"
-          rpy="0 0 ${M_PI/2.0}" />
-        <geometry>
-          <mesh filename="package://aroco_description/meshes/chassis.dae" />
-        </geometry>
-      </visual>
-      <!-- visual front steering -->
-      <mesh filename="package://aroco_description/meshes/wheel_steered.dae" />
-      <!-- visual rear steering -->
-      <mesh filename="package://aroco_description/meshes/wheel_steered.dae" />
-      <!-- visual front wheel -->
-      <mesh filename="package://aroco_description/meshes/wheel.dae" />
-      <!-- visual rear wheel -->
-      <mesh filename="package://aroco_description/meshes/wheel.dae" />
+      <xacro:chassis_visual />
+      <xacro:front_left_arm_visual />
+      <xacro:front_right_arm_visual />
+      <xacro:rear_left_arm_visual />
+      <xacro:rear_right_arm_visual />
+      <xacro:front_left_wheel_visual />
+      <xacro:front_right_wheel_visual />
+      <xacro:rear_left_wheel_visual />
+      <xacro:rear_right_wheel_visual />
     </xacro:chassis>
   </xacro:macro>
