Commit message: refactoring
Signed-off-by: Jean Laneurit <jean.laneurit@inrae.fr>

File: aroco_description/urdf/aroco.simulation.xacro (robot description, xacro)
@@ -4,5 +4,5 @@
     params="mode ros_prefix base_name controller_manager_config_yaml_file">
     <xacro:if value="${'simulation' in mode}">
-      <xacro:if value="${'gazebo' in  mode}">
+      <xacro:if value="${'gazebo_classic' in  mode}">
         <gazebo>
           <plugin filename="libgazebo_ros2_control.so" name="gazebo_ros2_control">
@@ -17,4 +17,18 @@
         </gazebo>
       </xacro:if>
+      <xacro:if value="${'gazebo_classic' not in  mode}">
+        <gazebo>
+          <plugin filename="gz_ros2_control-system"
+            name="gz_ros2_control::GazeboSimROS2ControlPlugin">
+            <robot_param>robot_description</robot_param>
+            <robot_param_node>ros2_control_description</robot_param_node>
+            <parameters>${controller_manager_config_yaml_file}</parameters>
+            <!-- <hold_joints>true</hold_joints> -->
+            <ros>
+              <namespace>${ros_prefix}${base_name}</namespace>
+            </ros>
+          </plugin>
+        </gazebo>
+      </xacro:if>
     </xacro:if>
   </xacro:macro>

File: aroco_description/urdf/visual/arms.xacro (robot description, xacro)
@@ -5,5 +5,6 @@
             <origin xyz="0.0 0.0 0.0" rpy="0 0 ${orientation}" />
             <geometry>
-                <mesh filename="package://aroco_description/meshes/wheel_steered.dae" />
+                <!-- <mesh filename="package://aroco_description/meshes/wheel_steered.dae" /> -->
+                <mesh filename="file://$(find aroco_description)/meshes/wheel_steered.dae" />
             </geometry>
             <material name=" grey">

File: aroco_description/urdf/visual/chassis.xacro (robot description, xacro)
@@ -6,5 +6,6 @@
                 rpy="0 0 ${M_PI/2.0}" />
             <geometry>
-                <mesh filename="package://aroco_description/meshes/chassis.dae" />
+                <!-- <mesh filename="package://aroco_description/meshes/chassis.dae" /> -->
+                <mesh filename="file://$(find aroco_description)/meshes/chassis.dae" />
             </geometry>
             <material name="grey">

File: aroco_description/urdf/visual/wheels.xacro (robot description, xacro)
@@ -5,5 +5,6 @@
             <origin xyz="0 0 0" rpy="0 ${orientation} 0" />
             <geometry>
-                <mesh filename="package://aroco_description/meshes/wheel.dae" />
+                <!-- <mesh filename="package://aroco_description/meshes/wheel.dae" /> -->
+                <mesh filename="file://$(find aroco_description)/meshes/wheel.dae" />
             </geometry>
             <material name="black">
